File: hardware/tinylab_09-03-16.sch (EAGLE design)
At the start: 148 parts, among them IC1 LM2575S, IC2 LM35CZ, IC3 LM358MX, IC4 MCP2300X/SO, IC5 LD117AS33TR, IC6 MAX7219CWG, J1 AVR_SPI_PRG_6NS, J2 POWER_JACKPTH_LOCK, K4 ZF112, M1 WIRELESS-NRF24L01, P1 P120PK, Q1 FDD4141 or FDD6637, Q3 BSS138, Q4 BSS138, SW1 ENCODER_SW1-PEC12, U1 LCD-16X2SILK, U2 24LC256, U5 USD-SOCKETNEW, Y1 16Mhz

Commit message: added resistor on lcd backlight led and done some  little changes.
Parts:
- added R13: 100R, SparkFun:RESISTOR0805-RES
- C21, C25: value 100n -> 100nF
- LED3, LED4, LED5, LED6: value (none) -> RED
- Q2: value (none) -> FDN340
- R46: value 30k civari -> 30k
- T1, T2, T3, T4: value (none) -> BC847
- U$15: value HEX_CONVERTER -> 74HC4050
- renumbered 74HC4050 to U$15, BC847 to T1, FDN340 to Q2
Connections:
- new net N$65: R13.1, U1.A
- net +5V: now also R13.2; no longer U1.A
Other:
- note added: "Designed by: Yusuf Gundogdu"
- note added: "Released under the GNU-GPL v2"
- note added: "Revised by: Okan Saracoglu"
- note added: "https://www.gnu.org/licenses/old-licenses/gpl-2.0.html"
- note added: "v1.3"
